File: etb-9201.sch (KiCad schematic (older format))
At the start: 5 parts, among them U1201 TLE9201SG

Commit message: #72
Changed lines of the file:
@@
 AR Path="/5DD457F9/5DD48EC1" Ref="C1202"  Part="1"
 AR Path="/5DDC2003/5DD48EC1" Ref="C1602"  Part="1"
-AR Path="/62471BCF/5DD48EC1" Ref="C28"  Part="1"
-AR Path="/6247AE9A/5DD48EC1" Ref="C31"  Part="1"
-F 0 "C31" H 3592 1171 50  0000 L CNN
+AR Path="/62471BCF/5DD48EC1" Ref="C1202"  Part="1"
+AR Path="/6247AE9A/5DD48EC1" Ref="C28"  Part="1"
+F 0 "C28" H 3592 1171 50  0000 L CNN
 F 1 "10n" H 3592 1080 50  0000 L CNN
 F 2 "Capacitor_SMD:C_0603_1608Metric" H 3500 1125 50  0001 C CNN
@@
 AR Path="/5DD457F9/5DD49883" Ref="C1203"  Part="1"
 AR Path="/5DDC2003/5DD49883" Ref="C1603"  Part="1"
-AR Path="/62471BCF/5DD49883" Ref="C29"  Part="1"
-AR Path="/6247AE9A/5DD49883" Ref="C32"  Part="1"
-F 0 "C32" H 3592 1621 50  0000 L CNN
+AR Path="/62471BCF/5DD49883" Ref="C1203"  Part="1"
+AR Path="/6247AE9A/5DD49883" Ref="C29"  Part="1"
+F 0 "C29" H 3592 1621 50  0000 L CNN
 F 1 "10n" H 3592 1530 50  0000 L CNN
 F 2 "Capacitor_SMD:C_0603_1608Metric" H 3500 1575 50  0001 C CNN
@@
 AR Path="/5DDC2003/5DD4C345" Ref="C1601"  Part="1"
 AR Path="/62471BCF/5DD4C345" Ref="C27"  Part="1"
-AR Path="/6247AE9A/5DD4C345" Ref="C30"  Part="1"
-F 0 "C30" H 2340 1096 50  0000 L CNN
+AR Path="/6247AE9A/5DD4C345" Ref="C1201"  Part="1"
+F 0 "C1201" H 2340 1096 50  0000 L CNN
 F 1 "10u" H 2340 1005 50  0000 L CNN
 F 2 "Capacitor_SMD:C_1206_3216Metric" H 2263 900 50  0001 C CNN
@@
 AR Path="/5DD457F9/5DF25274" Ref="R1001"  Part="1"
 AR Path="/5DDC2003/5DF25274" Ref="R1301"  Part="1"
-AR Path="/62471BCF/5DF25274" Ref="R48"  Part="1"
-AR Path="/6247AE9A/5DF25274" Ref="R49"  Part="1"
-F 0 "R49" V 1850 1450 50  0000 C CNN
+AR Path="/62471BCF/5DF25274" Ref="R1001"  Part="1"
+AR Path="/6247AE9A/5DF25274" Ref="R48"  Part="1"
+F 0 "R48" V 1850 1450 50  0000 C CNN
 F 1 "10k" V 1750 1450 50  0000 C CNN
 F 2 "Resistor_SMD:R_0402_1005Metric" V 1680 1450 50  0001 C CNN

Commit message: move diodes to front
Parts:
- C1202, C1203: PN CGA3E2X7R1H103M080AA -> (none)
Changed lines of the file:
@@
 $Descr A4 11693 8268
 encoding utf-8
-Sheet 19 19
+Sheet 18 19
 Title "rusEfi Proteus"
 Date "2020-01-17"
@@
 F 2 "Capacitor_SMD:C_0603_1608Metric" H 3500 1125 50  0001 C CNN
 F 3 "~" H 3500 1125 50  0001 C CNN
-F 4 "CGA3E2X7R1H103M080AA" H 3500 1125 50  0001 C CNN "PN"
+F 4 "" H 3500 1125 50  0001 C CNN "PN"
 F 5 "C57112" H 3500 1125 50  0001 C CNN "LCSC"
 F 6 "0" H 3500 1125 50  0001 C CNN "LCSC_ext"
@@
 F 2 "Capacitor_SMD:C_0603_1608Metric" H 3500 1575 50  0001 C CNN
 F 3 "~" H 3500 1575 50  0001 C CNN
-F 4 "CGA3E2X7R1H103M080AA" H 3500 1575 50  0001 C CNN "PN"
+F 4 "" H 3500 1575 50  0001 C CNN "PN"
 F 5 "C57112" H 3500 1575 50  0001 C CNN "LCSC"
 F 6 "0" H 3500 1575 50  0001 C CNN "LCSC_ext"
